File: pcb/atlas_tia/atlas_tia.kicad_sch (KiCad schematic)
At the start: 0 parts

Commit message: finished TIA layout
Parts:
- added C1: 0.5pF, Capacitor_SMD:C_0402_1005Metric, symbol Device:C
- added C2, C3: 100nF, Capacitor_SMD:C_0603_1608Metric, symbol Device:C
- added C4, C5: 10uF, Capacitor_SMD:C_1210_3225Metric, symbol Device:C
- added J1: TIA_LINK, Connector_JST:JST_GH_SM05B-GHS-TB_1x05-1MP_P1.25mm_Horizontal, symbol Connector_Generic:Conn_01x05
- added J2: TIP_CONTACT, atlas_parts_lib:TipContact_Pad_D0.8mm, symbol Connector_Generic:Conn_01x01
- added J3: SHIELD_CONTACT, Connector_Wire:SolderWirePad_1x01_SMD_1.5x3mm, symbol Connector_Generic:Conn_01x01
- added R1: 100M, Resistor_SMD:R_1206_3216Metric, symbol Device:R
- added R2: 220, Resistor_SMD:R_0603_1608Metric, symbol Device:R
- added R3, R4: 10, Resistor_SMD:R_0603_1608Metric, symbol Device:R
- added TP1, TP2, TP3, TP4, TP5: TestPoint, TestPoint:TestPoint_Pad_D1.0mm, symbol Connector:TestPoint
- added U1: OPA828IDR, Package_SO:SOIC-8_3.9x4.9mm_P1.27mm, symbol atlas_parts_lib:OPA828IDR
Connections:
- new net +15V: J1.4 (Pin_4), R3.1
- new net -15V: J1.5 (Pin_5), R4.1
- new net CHASSIS: J3.1 (Pin_1)
- new net GNDA: C2.2, C3.2, C4.2, C5.2, J1.2 (Pin_2), J1.3 (Pin_3), TP5.1, U1.3 (+)
- new net TIA_OUT: J1.1 (Pin_1), R2.2, TP2.1
- new net TIA_RAW: C1.2, R1.2, R2.1, TP1.1, U1.6
- new net TIP_IN: C1.1, J2.1 (Pin_1), R1.1, U1.2 (-)
- new net VCC_TIA: C2.1, C4.1, R3.2, TP3.1, U1.7 (V+)
- new net VEE_TIA: C3.1, C5.1, R4.2, TP4.1, U1.4 (V-)
Other:
- note added: "CHASSIS bond pending system ground review. No GNDA-to-chassis bond is fitted here."
- note added: "External supply declarations: incoming rails, filtered rails and analog return."
- note added: "J1.2: quiet ground sense; J1.3: power return. Route separately to the converter."

Commit message: final save + updated README
Other:
- note removed: "CHASSIS bond pending system ground review. No GNDA-to-chassis bond is fitted here."
- note removed: "External supply declarations: incoming rails, filtered rails and analog return."
- note removed: "J1.2: quiet ground sense; J1.3: power return. Route separately to the converter."
- moved on the sheet: C1, C2, C3, C4, C5, R1, R2, R3, R4
