File: pcb/atlas_tia/atlas_tia.kicad_sch (KiCad schematic)
At the start: 18 parts, among them J1 TIA_LINK, J2 TIP_CONTACT, J3 SHIELD_CONTACT, U1 OPA828IDR

Commit message: TIA layout updates, guard footprints and LTspice compensation study
- Update TIA schematic, board and project
- Add guard-ring variants of C_0603, R_1206 and SOIC-8 footprints to atlas_parts_lib
- Add LTspice TIA netlists (proxy and TI OPAx828 model), analysis scripts and sweep results

Co-Authored-By: Claude Opus 5.5 <noreply@anthropic.com>
Parts:
- C1: value 0.5pF -> 0.2pF; footprint Capacitor_SMD:C_0402_1005Metric -> atlas_parts_lib:C_0603_1608Metric_Guard; MPN (none) -> CQ0603BRNPO9BNR20; Manufacturer (none) -> YAGEO; Tolerance (none) -> ±0.1pF
- J2: footprint atlas_parts_lib:TipContact_Pad_D0.8mm -> Connector_Wire:SolderWirePad_1x01_SMD_1x2mm
- R1: footprint Resistor_SMD:R_1206_3216Metric -> atlas_parts_lib:R_1206_3216Metric_Guard
- U1: footprint Package_SO:SOIC-8_3.9x4.9mm_P1.27mm -> atlas_parts_lib:SOIC-8_3.9x4.9mm_P1.27mm_Guard
Connections:
- net GNDA: now also U1.1 (NC)
Other:
- note added: "U1.1: grounded PCB guard; NC internally"
Changed lines of the file:
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@@
 			)
 		)
-		(property "Footprint" "atlas_parts_lib:TipContact_Pad_D0.8mm"
+		(property "Footprint" "Connector_Wire:SolderWirePad_1x01_SMD_1x2mm"
 			(at 88.9 30.48 0)
 			(hide yes)
@@
 			)
 		)
-		(property "Footprint" "Resistor_SMD:R_1206_3216Metric"
+		(property "Footprint" "atlas_parts_lib:R_1206_3216Metric_Guard"
 			(at 199.39 86.868 90)
 			(hide yes)
@@
 			)
 		)
-		(property "Footprint" "Package_SO:SOIC-8_3.9x4.9mm_P1.27mm"
+		(property "Footprint" "atlas_parts_lib:SOIC-8_3.9x4.9mm_P1.27mm_Guard"
 			(at 172.72 49.53 0)
 			(hide yes)
@@
 			)
 		)
-		(property "Value" "0.5pF"
+		(property "Value" "0.2pF"
 			(at 133.35 78.7399 0)
 			(show_name no)
@@
 			)
 		)
-		(property "Footprint" "Capacitor_SMD:C_0402_1005Metric"
+		(property "Footprint" "atlas_parts_lib:C_0603_1608Metric_Guard"
 			(at 130.5052 81.28 0)
 			(hide yes)
@@
 			)
 		)
-		(property "Datasheet" ""
+		(property "Datasheet" "https://yageogroup.com/content/datasheet/asset/file/UPY-HIGH_Q_NP0_16V-TO-500V"
 			(at 129.54 77.47 0)
 			(hide yes)
@@
 		)
 		(property "Dielectric" "C0G/NP0"
+			(at 129.54 77.47 0)
+			(hide yes)
+			(show_name no)
+			(do_not_autoplace no)
+			(effects
+				(font
+					(size 1.27 1.27)
+				)
+			)
+		)
+		(property "Tolerance" "±0.1pF"
+			(at 129.54 77.47 0)
+			(hide yes)
+			(show_name no)
+			(do_not_autoplace no)
+			(effects
+				(font
+					(size 1.27 1.27)
+				)
+			)
+		)
+		(property "Manufacturer" "YAGEO"
+			(at 129.54 77.47 0)
+			(hide yes)
+			(show_name no)
+			(do_not_autoplace no)
+			(effects
+				(font
+					(size 1.27 1.27)
+				)
+			)
+		)
+		(property "MPN" "CQ0603BRNPO9BNR20"
 			(at 129.54 77.47 0)
 			(hide yes)
@@
 	)
 	(embedded_fonts no)
+ (wire (pts (xy 172.72 41.91) (xy 172.72 36.83))
+  (stroke (width 0) (type default)))
+ (global_label "GNDA" (shape input) (at 172.72 36.83 90)
+  (effects (font (size 1.27 1.27)) (justify left)))
+ (text "U1.1: grounded PCB guard; NC internally" (at 177.8 33.02 0)
+  (effects (font (size 1 1)) (justify left bottom)))
 )
