File: pcb/atlas_tia/atlas_tia.kicad_pcb (KiCad board)
At the start: 2 copper layers, 17 parts, among them J1 TIA_LINK, J3 SHIELD_CONTACT, U1 OPA828IDR

Commit message: edited gitignore; finished TIA layout
Parts:
- added J2: TIP_CONTACT, atlas_parts_lib:TipContact_Pad_D0.8mm, F.Cu at (135.2, 108.1)
- moved J3 13.0 mm to (120.3, 107.7)
- moved R1 13.0 mm to (131.2, 108.6)
- moved C1 13.0 mm to (117.1, 109.1)
- moved C4 13.0 mm to (125.6, 102.5)
- moved C5 13.0 mm to (125.6, 106.7)
- moved R2 13.0 mm to (120.8, 99.2)
- moved R4 13.0 mm to (120.8, 104.2)
- moved TP1 13.0 mm to (117.2, 94.4)
- moved TP2 13.0 mm to (117.2, 97.5)
- moved U1 13.0 mm to (132.6, 103.7)
- moved C2 13.0 mm to (120.8, 94.2)
- moved C3 13.0 mm to (120.8, 96.7)
- moved J1 13.0 mm to (128.6, 96.6)
- moved R3 13.0 mm to (120.8, 101.7)
- moved TP3 13.0 mm to (117.2, 100.5)
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