File: pcb/atlas_psu/atlas_psu.kicad_sch (KiCad schematic)
At the start: 0 parts

Commit message: PSU schematic: add BOM fields, design notes and power net class; ignore review docs
- Add Manufacturer/MPN/LCSC/Tolerance/Power/Voltage fields from the design plan
- Add title block and design/assembly notes to the PSU sheet
- Add Power net class for AC, RAW, REG, SYS and PSU_0V nets
- Import PSU footprints into the board
- Ignore *_REVIEW.md, *_EVALUATION.md and PCB routing_review snapshots

Co-Authored-By: Claude Opus 5.5 <noreply@anthropic.com>
Parts:
- added C1, C2: 4700uF, Capacitor_THT:CP_Radial_D30.0mm_P10.00mm_SnapIn, symbol Device:C_Polarized
- added C10, C11, C4, C6, C8, C9: 10uF, Capacitor_SMD:CP_Elec_6.3x5.4_Nichicon, symbol Device:C_Polarized
- added C12, C13, C3, C5: 100nF, Capacitor_SMD:C_0603_1608Metric, symbol Device:C
- added C7: 47uF, Capacitor_SMD:CP_Elec_6.3x7.7, symbol Device:C_Polarized
- added D1, D2, D3, D4, D5, D6, D7, D8, D9: M7, Diode_SMD:D_SMA, symbol Device:D
- added D10: GBU4M-E3/51, Diode_THT:Diode_Bridge_Vishay_GBU, symbol Diode_Bridge:GBU4M
- added J1: SECONDARY_AC, TerminalBlock_Phoenix:TerminalBlock_Phoenix_MKDS-1,5-4-5.08_1x04_P5.08mm_Horizontal, symbol Connector_Generic:Conn_01x04
- added J2: NORMAL_SOURCE, Connector_JST:JST_XH_B4B-XH-A_1x04_P2.50mm_Vertical, symbol Connector_Generic:Conn_01x04
- added J3: SYSTEM_FEED, Connector_JST:JST_XH_B4B-XH-A_1x04_P2.50mm_Vertical, symbol Connector_Generic:Conn_01x04
- added J4: ANALOG_POWER, Connector_JST:JST_XH_B4B-XH-A_1x04_P2.50mm_Vertical, symbol Connector_Generic:Conn_01x04
- added J5: STACK_POWER, Connector_JST:JST_XH_B3B-XH-A_1x03_P2.50mm_Vertical, symbol Connector_Generic:Conn_01x03
- added J6: PSU_STATUS, Connector_JST:JST_GH_SM03B-GHS-TB_1x03-1MP_P1.25mm_Horizontal, symbol Connector_Generic:Conn_01x03
- added J7: CHASSIS_CONTACT, Connector_Wire:SolderWirePad_1x01_SMD_1.5x3mm, symbol Connector_Generic:Conn_01x01
- added R1, R3, R5: 110, Resistor_SMD:R_0603_1608Metric, symbol Device:R
- added R10, R12, R14, R18: 10k, Resistor_SMD:R_0603_1608Metric, symbol Device:R
- added R11, R9: 45k3, Resistor_SMD:R_0603_1608Metric, symbol Device:R
- added R13: 16k2, Resistor_SMD:R_0603_1608Metric, symbol Device:R
- added R15, R16: 1k8, Resistor_SMD:R_1206_3216Metric, symbol Device:R
- added R17: 470, Resistor_SMD:R_1206_3216Metric, symbol Device:R
- added R19: 100, Resistor_SMD:R_0603_1608Metric, symbol Device:R
- added R2, R4: 1k21, Resistor_SMD:R_0805_2012Metric, symbol Device:R
- added R6: 549, Resistor_SMD:R_0805_2012Metric, symbol Device:R
- added R7, R8: 10k, Resistor_SMD:R_2010_5025Metric, symbol Device:R
- added TP1, TP10, TP2, TP3, TP4, TP5, TP6, TP7, TP8, TP9: TestPoint, TestPoint:TestPoint_Pad_D1.0mm, symbol Connector:TestPoint
- added U1, U3: LM317T, Package_TO_SOT_THT:TO-220-3_Vertical, symbol Regulator_Linear:LM317_TO-220
- added U2: LM337T, Package_TO_SOT_THT:TO-220-3_Vertical, symbol Regulator_Linear:LM337_TO220
- added U4, U5, U6: TL431BIDBZR, Package_TO_SOT_SMD:SOT-23, symbol Reference_Voltage:TL431DBZ
- added U7, U8, U9: LTV-817S-TA1-D, Package_DIP:SMDIP-4_W9.53mm, symbol Isolator:LTV-817S
Connections:
- new net AC_A: D10.2, J1.1 (Pin_1)
- new net AC_B: D10.3, J1.4 (Pin_4)
- new net ADJ_AUX: C11.1, D6.2 (A), R5.2, R6.1, U3.1 (ADJ)
- new net ADJ_N: C10.2, D4.1 (K), R3.2, R4.1, U2.1 (ADJ)
- new net ADJ_P: C9.1, D2.2 (A), R1.2, R2.1, U1.1 (ADJ)
- new net CHASSIS: J7.1 (Pin_1)
- new net DET_A_K: U6.1 (K), U9.2
- new net DET_A_REF: R13.2, R14.1, U6.2 (REF)
- new net DET_N_K: U5.1 (K), U8.2
- new net DET_N_REF: R11.2, R12.1, U5.2 (REF)
- new net DET_P_K: U4.1 (K), U7.2
- new net DET_P_REF: R10.1, R9.2, U4.2 (REF)
- new net LED_A_A: R17.2, U9.1
- new net LED_N_A: R16.2, U8.1
- new net LED_P_A: R15.2, U7.1
- new net OK_FEED: R19.2, U7.4
- new net OK_LINK_1: U7.3, U8.4
- new net OK_LINK_2: U8.3, U9.4
- new net PSU_0V: C1.2, C10.1, C11.2, C12.2, C13.2, C2.1, C3.2, C4.1, C5.2, C6.2, C7.1, C8.2, C9.2, D7.2 (A), D8.1 (K), D9.2 (A), J1.2 (Pin_2), J1.3 (Pin_3), J2.2 (Pin_2), R2.2, R4.2, R6.2, R7.2, R8.1, TP3.1
- new net PSU_VALID: J6.2 (Pin_2), R18.1, TP10.1, U9.3
- new net RAW_N: C2.2, C4.2, D10.4 (-), D3.2 (A), R8.2, TP2.1, U2.2 (VI)
- new net RAW_P: C1.1, C3.1, C5.1, D1.1 (K), D10.1 (+), D5.1 (K), R7.1, TP1.1, U1.3 (VI), U3.3 (VI)
- new net REG_AUX: C13.1, C8.1, D5.2 (A), D6.1 (K), D9.1 (K), J2.4 (Pin_4), R5.1, TP6.1, U3.2 (VO)
- new net REG_N15: C7.2, D3.1 (K), D4.2 (A), D8.2 (A), J2.3 (Pin_3), R3.1, TP5.1, U2.3 (VO)
- new net REG_P15: C12.1, C6.1, D1.2 (A), D2.1 (K), D7.1 (K), J2.1 (Pin_1), R1.1, TP4.1, U1.2 (VO)
- new net STATUS_0V: J6.3 (Pin_3), R18.2
- new net STATUS_3V3: J6.1 (Pin_1), R19.1
- new net SYS_0V: J3.2 (Pin_2), J4.2 (Pin_2), J5.2 (Pin_2), R10.2, R11.1, R14.2, R16.1, U4.3 (A), U6.3 (A)
- new net SYS_AUX: J3.4 (Pin_4), J4.4 (Pin_4), R13.1, R17.1, TP9.1
- new net SYS_N15: J3.3 (Pin_3), J4.3 (Pin_3), J5.3 (Pin_3), R12.2, TP8.1, U5.3 (A)
- new net SYS_P15: J3.1 (Pin_1), J4.1 (Pin_1), J5.1 (Pin_1), R15.1, R9.1, TP7.1
Other:
- note added: "1. OFF-BOARD SOURCE: T1 (2 x 18 V AC, 30 VA) and both secondary fuses FSEC1/FSEC2 are off this PCB. Mains primary, inlet, primary fuse, switch and PE bonding stay in the enclosure; none of it reaches this board. Phase the windings so A2-B1 gives ~36 V AC between J1.1 and J1.4; check before connecting the bridge. 2. SOURCE SELECTION: J2 (NORMAL_SOURCE) reaches J3 (SYSTEM_FEED) ONLY through the rem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"
- note added: "DESIGN AND ASSEMBLY NOTES"
- title: (none) -> ATLAS PSU: linear +/-15 V and +7.5 V supply
